Commit message: rename to eddie, update dependent repo links

File: eddie_gazebo/urdf/eddie.urdf (robot description, URDF)
Before this commit: robot freddy, 57 links, 56 joints
Links:
- removed link freddy_base_link
- removed link freddy_torso_link
- removed link freddy_torso_shoulder_left_arm_attach_link
- removed link freddy_torso_shoulder_left_link
- removed link freddy_torso_shoulder_right_arm_attach_link
- removed link freddy_torso_shoulder_right_link
- added link eddie_base_link, mass 40.0; collision box size=0.635 0.582 0.1; collision box size=0.635 0.582 0.12
- added link eddie_torso_link, mass 40.0; collision box size=0.19 0.4 0.3; visual box size=0.19 0.4 0.3
- added link eddie_torso_shoulder_left_arm_attach_link
- added link eddie_torso_shoulder_left_link, mass 40.0; collision box size=0.02 0.2 0.2; visual box size=0.02 0.2 0.2
- added link eddie_torso_shoulder_right_arm_attach_link
- added link eddie_torso_shoulder_right_link, mass 40.0; collision box size=0.02 0.2 0.2; visual box size=0.02 0.2 0.2
- link base_laser_back_link: geometry collision mesh filename=package://eddie_base_description/meshes/sensors/hokuyo_conv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; visual mesh filename=package://eddie_base_description/meshes/sensors/hokuyo.dae
- link base_laser_front_link: geometry collision mesh filename=package://eddie_base_description/meshes/sensors/hokuyo_conv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; visual mesh filename=package://eddie_base_description/meshes/sensors/hokuyo.dae
- link kinova_left_base_link: geometry collision mesh filename=file:///home/shinas/ros2/eddie/install/kortex_description/s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; visual mesh filename=file:///home/shinas/ros2/eddie/install/kortex_description/s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
- link kinova_left_bracelet_link: geometry collision mesh filename=file:///home/shinas/ros2/eddie/install/kortex_description/s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; visual mesh filename=file:///home/shinas/ros2/eddie/install/kortex_description/s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
- link kinova_left_forearm_link: geometry collision mesh filename=file:///home/shinas/ros2/eddie/install/kortex_description/s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; visual mesh filename=file:///home/shinas/ros2/eddie/install/kortex_description/s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
- link kinova_left_half_arm_1_link: geometry collision mesh filename=file:///home/shinas/ros2/eddie/install/kortex_description/s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; visual mesh filename=file:///home/shinas/ros2/eddie/install/kortex_description/s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
- link kinova_left_half_arm_2_link: geometry collision mesh filename=file:///home/shinas/ros2/eddie/install/kortex_description/s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; visual mesh filename=file:///home/shinas/ros2/eddie/install/kortex_description/s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
- link kinova_left_robotiq_85_base_link: geometry collision mesh filename=file:///home/shinas/ros2/eddie/install/robotiq_description/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; visual mesh filename=file:///home/shinas/ros2/eddie/install/robotiq_description/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
- link kinova_left_robotiq_85_left_finger_link: geometry collision mesh filename=file:///home/shinas/ros2/eddie/install/robotiq_description/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; visual mesh filename=file:///home/shinas/ros2/eddie/install/robotiq_description/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
- link kinova_left_robotiq_85_left_finger_tip_link: geometry collision mesh filename=file:///home/shinas/ros2/eddie/install/robotiq_description/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; visual mesh filename=file:///home/shinas/ros2/eddie/install/robotiq_description/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
- link kinova_left_robotiq_85_left_inner_knuckle_link: geometry collision mesh filename=file:///home/shinas/ros2/eddie/install/robotiq_description/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; visual mesh filename=file:///home/shinas/ros2/eddie/install/robotiq_description/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
- link kinova_left_robotiq_85_left_knuckle_link: geometry collision mesh filename=file:///home/shinas/ros2/eddie/install/robotiq_description/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; visual mesh filename=file:///home/shinas/ros2/eddie/install/robotiq_description/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
- link kinova_left_robotiq_85_right_finger_link: geometry collision mesh filename=file:///home/shinas/ros2/eddie/install/robotiq_description/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; visual mesh filename=file:///home/shinas/ros2/eddie/install/robotiq_description/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
- link kinova_left_robotiq_85_right_finger_tip_link: geometry collision mesh filename=file:///home/shinas/ros2/eddie/install/robotiq_description/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; visual mesh filename=file:///home/shinas/ros2/eddie/install/robotiq_description/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
- link kinova_left_robotiq_85_right_inner_knuckle_link: geometry collision mesh filename=file:///home/shinas/ros2/eddie/install/robotiq_description/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; visual mesh filename=file:///home/shinas/ros2/eddie/install/robotiq_description/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
- link kinova_left_robotiq_85_right_knuckle_link: geometry collision mesh filename=file:///home/shinas/ros2/eddie/install/robotiq_description/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; visual mesh filename=file:///home/shinas/ros2/eddie/install/robotiq_description/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
- link kinova_left_shoulder_link: geometry collision mesh filename=file:///home/shinas/ros2/eddie/install/kortex_description/s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; visual mesh filename=file:///home/shinas/ros2/eddie/install/kortex_description/s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
- link kinova_left_spherical_wrist_1_link: geometry collision mesh filename=file:///home/shinas/ros2/eddie/install/kortex_description/s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; visual mesh filename=file:///home/shinas/ros2/eddie/install/kortex_description/s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
- link kinova_left_spherical_wrist_2_link: geometry collision mesh filename=file:///home/shinas/ros2/eddie/install/kortex_description/s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; visual mesh filename=file:///home/shinas/ros2/eddie/install/kortex_description/s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
- link kinova_right_base_link: geometry collision mesh filename=file:///home/shinas/ros2/eddie/install/kortex_description/s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; visual mesh filename=file:///home/shinas/ros2/eddie/install/kortex_description/s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
- link kinova_right_bracelet_link: geometry collision mesh filename=file:///home/shinas/ros2/eddie/install/kortex_description/s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; visual mesh filename=file:///home/shinas/ros2/eddie/install/kortex_description/s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
- link kinova_right_forearm_link: geometry collision mesh filename=file:///home/shinas/ros2/eddie/install/kortex_description/s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; visual mesh filename=file:///home/shinas/ros2/eddie/install/kortex_description/s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
- link kinova_right_half_arm_1_link: geometry collision mesh filename=file:///home/shinas/ros2/eddie/install/kortex_description/s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; visual mesh filename=file:///home/shinas/ros2/eddie/install/kortex_description/s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
- link kinova_right_half_arm_2_link: geometry collision mesh filename=file:///home/shinas/ros2/eddie/install/kortex_description/s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; visual mesh filename=file:///home/shinas/ros2/eddie/install/kortex_description/s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
- link kinova_right_robotiq_85_base_link: geometry collision mesh filename=file:///home/shinas/ros2/eddie/install/robotiq_description/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; visual mesh filename=file:///home/shinas/ros2/eddie/install/robotiq_description/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
- link kinova_right_robotiq_85_left_finger_link: geometry collision mesh filename=file:///home/shinas/ros2/eddie/install/robotiq_description/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; visual mesh filename=file:///home/shinas/ros2/eddie/install/robotiq_description/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
- link kinova_right_robotiq_85_left_finger_tip_link: geometry collision mesh filename=file:///home/shinas/ros2/eddie/install/robotiq_description/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; visual mesh filename=file:///home/shinas/ros2/eddie/install/robotiq_description/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
- link kinova_right_robotiq_85_left_inner_knuckle_link: geometry collision mesh filename=file:///home/shinas/ros2/eddie/install/robotiq_description/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; visual mesh filename=file:///home/shinas/ros2/eddie/install/robotiq_description/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
- link kinova_right_robotiq_85_left_knuckle_link: geometry collision mesh filename=file:///home/shinas/ros2/eddie/install/robotiq_description/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; visual mesh filename=file:///home/shinas/ros2/eddie/install/robotiq_description/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
- link kinova_right_robotiq_85_right_finger_link: geometry collision mesh filename=file:///home/shinas/ros2/eddie/install/robotiq_description/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; visual mesh filename=file:///home/shinas/ros2/eddie/install/robotiq_description/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
- link kinova_right_robotiq_85_right_finger_tip_link: geometry collision mesh filename=file:///home/shinas/ros2/eddie/install/robotiq_description/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; visual mesh filename=file:///home/shinas/ros2/eddie/install/robotiq_description/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
- link kinova_right_robotiq_85_right_inner_knuckle_link: geometry collision mesh filename=file:///home/shinas/ros2/eddie/install/robotiq_description/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; visual mesh filename=file:///home/shinas/ros2/eddie/install/robotiq_description/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
- link kinova_right_robotiq_85_right_knuckle_link: geometry collision mesh filename=file:///home/shinas/ros2/eddie/install/robotiq_description/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; visual mesh filename=file:///home/shinas/ros2/eddie/install/robotiq_description/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
- link kinova_right_shoulder_link: geometry collision mesh filename=file:///home/shinas/ros2/eddie/install/kortex_description/s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; visual mesh filename=file:///home/shinas/ros2/eddie/install/kortex_description/s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
- link kinova_right_spherical_wrist_1_link: geometry collision mesh filename=file:///home/shinas/ros2/eddie/install/kortex_description/s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; visual mesh filename=file:///home/shinas/ros2/eddie/install/kortex_description/s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
- link kinova_right_spherical_wrist_2_link: geometry collision mesh filename=file:///home/shinas/ros2/eddie/install/kortex_description/s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; visual mesh filename=file:///home/shinas/ros2/eddie/install/kortex_description/s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
Joints:
- removed joint freddy_base_joint
- removed joint freddy_torso_joint
- removed joint freddy_torso_shoulder_left_arm_joint
- removed joint freddy_torso_shoulder_left_joint
- removed joint freddy_torso_shoulder_right_arm_joint
- removed joint freddy_torso_shoulder_right_joint
- added joint eddie_base_joint: type fixed, parent base_link, child eddie_base_link, origin xyz=0.0 0.0 0.0 rpy=0.0 0.0 0.0
- added joint eddie_torso_joint: type fixed, parent base_link, child eddie_torso_link, origin xyz=-0.20249999999999999 0 0.37 rpy=0 0 0
- added joint eddie_torso_shoulder_left_arm_joint: type fixed, parent eddie_torso_shoulder_left_link, child eddie_torso_shoulder_left_arm_attach_link, origin xyz=0 0.1 0.1 rpy=3.14159 -1.5708 0
- added joint eddie_torso_shoulder_left_joint: type fixed, parent eddie_torso_link, child eddie_torso_shoulder_left_link, origin xyz=0.085 0 0.27 rpy=0. 0.1309 0.7853982
- added joint eddie_torso_shoulder_right_arm_joint: type fixed, parent eddie_torso_shoulder_right_link, child eddie_torso_shoulder_right_arm_attach_link, origin xyz=0 -0.1 0.1 rpy=3.14159 -1.5708 0
- added joint eddie_torso_shoulder_right_joint: type fixed, parent eddie_torso_link, child eddie_torso_shoulder_right_link, origin xyz=0.085 0 0.27 rpy=0 0.1309 -0.7853982
- joint base_laser_back_joint: parent freddy_base_link -> eddie_base_link
- joint base_laser_front_joint: parent freddy_base_link -> eddie_base_link
- joint kinova_left_base_joint: parent freddy_torso_shoulder_left_arm_attach_link -> eddie_torso_shoulder_left_arm_attach_link
- joint kinova_right_base_joint: parent freddy_torso_shoulder_right_arm_attach_link -> eddie_torso_shoulder_right_arm_attach_link
- joint left_back_wheel_joint: parent freddy_base_link -> eddie_base_link
- joint left_front_wheel_joint: parent freddy_base_link -> eddie_base_link
- joint right_back_wheel_joint: parent freddy_base_link -> eddie_base_link
- joint right_front_wheel_joint: parent freddy_base_link -> eddie_base_link
